Commit message: add lamp and camera to xacro

File: workspaceRos/src/phantomx/phantomx_description/urdf/phantomx_urdf.xacro (robot description, xacro)
@@ -4,4 +4,10 @@
     <xacro:property name="thigh_offset_y" value="-0.0645"/>
     <xacro:property name="thigh_offset_z" value="-0.0145"/>
+    <xacro:property name="PI" value="3.1415926535897931"/>
+    <xacro:macro name = "sphere_geometry" params= "radius">
+        <geometry>
+            <sphere radius = "${radius}"/>
+        </geometry>
+    </xacro:macro>
     <xacro:macro name="phantomx" params="parent *origin">
         <joint name="j_phantomx_attachment" type="fixed">
@@ -43,4 +49,60 @@
         <xacro:leg_l xyz="-0.1248 0.06164  0.001116" rpy="0 4.7123 3.9269908169872414" suffix="lr"/>
     </xacro:macro>
+    <link name = "camera">
+        <visual>
+            <xacro:sphere_geometry radius = "0.02"/>
+        </visual>
+        <collision>
+            <xacro:sphere_geometry radius = "0.02"/>
+        </collision>
+        <inertial>
+            <mass value="0.05"/>
+            <inertia
+            ixx="0.01" ixy="0.0" ixz="0.0"
+            iyy="0.01" iyz="0.0"
+            izz="0.01"/>
+        </inertial>
+    </link>
+    <gazebo reference="camera">
+        <sensor type="camera" name="camera_vision">
+        <update_rate>30.0</update_rate>
+        <camera name="head">
+            <horizontal_fov>1.57</horizontal_fov>
+            <image>
+                <width>800</width>
+                <height>800</height>
+                <format>R8G8B8</format>
+            </image>
+            <clip>
+                <near>0.02</near>
+                <far>300</far>
+            </clip>
+            <noise>
+                <type>gaussian</type>
+                <mean>0.0</mean>
+                <stddev>0.007</stddev>
+            </noise>
+        </camera>
+            <plugin name="camera_controller" filename="libgazebo_ros_camera.so">
+                <alwaysOn>true</alwaysOn>
+                <updateRate>0.0</updateRate>
+                <cameraName>camera</cameraName>
+                <imageTopicName>image_raw</imageTopicName>
+                <cameraInfoTopicName>camera_info</cameraInfoTopicName>
+                <frameName>camera_frame</frameName>
+                <hackBaseline>0.07</hackBaseline>
+                <distortionK1>0.0</distortionK1>
+                <distortionK2>0.0</distortionK2>
+                <distortionK3>0.0</distortionK3>
+                <distortionT1>0.0</distortionT1>
+                <distortionT2>0.0</distortionT2>
+            </plugin>
+        </sensor>
+    </gazebo>
+    <joint name="lidar_to_camera" type="fixed">
+        <parent link="lidar"/>
+        <child link="camera"/>
+        <origin xyz="0.035 0 0.04" rpy="0 0 0"/>
+    </joint>
      <link name="lidar">
        <visual>
@@ -100,5 +162,5 @@
             <origin xyz="0 0 0.05"/>
     </joint>
-   <gazebo>
+    <gazebo>
      <plugin name="imu_plugin" filename="libgazebo_ros_imu.so">
        <alwaysOn>true</alwaysOn>
@@ -109,5 +171,27 @@
        <updateRate>20.0</updateRate>
      </plugin>
-   </gazebo>
+    </gazebo>
+    <link name="lamp">
+       <visual>
+        <geometry>
+         <cylinder length="0.01" radius="0.005"/>
+        </geometry>
+       </visual>
+      <collision>
+        <geometry>
+         <cylinder length="0.01" radius="0.005"/>
+        </geometry>
+      </collision>
+      <inertial>
+       <mass value="0.005"/>
+       <origin rpy="0 0 0" xyz="0 0 0.1"/>
+      <inertia ixx="0.0395416666667" ixy="0" ixz="0" iyy="0.106208333333" iyz="0" izz="0.106208333333"/>
+      </inertial>
+     </link>
+    <joint name="camera_to_lamp" type="fixed">
+            <parent link="camera"/>
+            <child link="lamp"/>
+            <origin xyz="0 0 0.025" rpy="0 ${-PI/2} 0" />
+    </joint>
      <xacro:macro name="leg_l" params="xyz rpy suffix">
         <link name="c1_${suffix}">

Commit message: change camera axis

File: workspaceRos/src/phantomx/phantomx_description/urdf/phantomx_urdf.xacro (robot description, xacro)
@@ -103,5 +103,5 @@
         <parent link="lidar"/>
         <child link="camera"/>
-        <origin xyz="0.035 0 0.04" rpy="0 0 0"/>
+        <origin xyz="0.0 0.035 0.04" rpy="0 0 1.57"/>
     </joint>
      <link name="lidar">

Commit message: change camera orientation

File: workspaceRos/src/phantomx/phantomx_description/urdf/phantomx_urdf.xacro (robot description, xacro)
@@ -103,5 +103,5 @@
         <parent link="lidar"/>
         <child link="camera"/>
-        <origin xyz="0.0 0.035 0.04" rpy="0 0 1.57"/>
+        <origin xyz="0.0 -0.035 0.04" rpy="0 0 -1.57"/>
     </joint>
      <link name="lidar">

Commit message: change camera orientation

File: workspaceRos/src/phantomx/phantomx_description/urdf/phantomx_urdf.xacro (robot description, xacro)
@@ -103,5 +103,5 @@
         <parent link="lidar"/>
         <child link="camera"/>
-        <origin xyz="0.0 -0.035 0.04" rpy="0 0 -1.57"/>
+        <origin xyz="0.0 -0.035 0.04" rpy="0 -0.5 -1.57"/>
     </joint>
      <link name="lidar">
